File: dpad/dpad.kicad_pcb (KiCad board)
At the start: 2 copper layers, 9 parts, among them J6 Conn_01x05_Socket, SW1 SW_Push_Dual, SW2 SW_Push_Dual, SW3 SW_Push_Dual, SW4 SW_Push_Dual

Commit message: dpad v0
Parts:
- J1: renamed from J6; footprint Connector_PinHeader_1.00mm:PinHeader_1x05_P1.00mm_Vertical -> Connector_PinHeader_2.54mm:PinHeader_1x05_P2.54mm_Vertical
- SW1, SW2, SW3, SW4: footprint Button_Switch_THT:SW_PUSH-12mm -> Button_Switch_THT:SW_PUSH_6mm
- moved SW4 27.4 mm to (89.5, 46.9), turned to -45 degrees
- moved J1 23.9 mm to (78.0, 66.5), turned to -90 degrees
- moved SW1 20.3 mm to (71.8, 51.5), turned to 45 degrees
- moved SW2 14.2 mm to (86.1, 59.9), turned to 180 degrees
- moved H3 13.6 mm to (98.0, 38.2), turned to 90 degrees
- moved H4 13.5 mm to (98.2, 70.2), turned to 90 degrees
- moved SW3 13.4 mm to (86.2, 44.9), turned to 180 degrees
- moved H1 10.5 mm to (67.2, 38.2), turned to -90 degrees
- moved H2 10.5 mm to (67.2, 70.2), turned to -90 degrees
- renumbered H5 to H1, H6 to H2, H7 to H3, H8 to H4
Routing:
- net D3: track 30.8 -> 52.5 mm
- net D4: track 10.7 -> 25.0 mm
- net D2: track 16.4 -> 13.5 mm
- net D1: track 21.5 -> 24.1 mm
- added copper zone on B.Cu, net GND
Other:
- board outline added: 40 x 40 mm
- board text added: "${COMPANY} ${ISSUE_DATE} D-Pad V${REVISION}"
- board text added: "GND"
- board text added: "JLCJLCJLCJLC"
- board text added: "SW1"
- board text added: "SW2"
- board text added: "SW3"
- board text added: "SW4"
- board text added: "https://www.gamecraft.it/"

Commit message: dpad v1
Parts:
- H1, H2, H3, H4: footprint MountingHole:MountingHole_3.2mm_M3_Pad -> MountingHole:MountingHole_2.2mm_M2_Pad
- moved H2 3.35 mm to (70.4, 71.2)
- moved H1 3.24 mm to (70.4, 38.7)
- moved H4 2.97 mm to (95.4, 71.2)
- moved H3 2.69 mm to (95.4, 38.7)
Routing:
- net D3: track 52.5 -> 49.4 mm
Other:
- board size 40 x 40 mm -> 31 x 39 mm
