File: dpad/dpad.kicad_sch (KiCad schematic)
At the start: 9 parts, among them J6 Conn_01x05_Socket, SW1 SW_Push_Dual, SW2 SW_Push_Dual, SW3 SW_Push_Dual, SW4 SW_Push_Dual

Commit message: dpad v0
Parts:
- J1: renamed from J6; footprint Connector_PinHeader_1.00mm:PinHeader_1x05_P1.00mm_Vertical -> Connector_PinHeader_2.54mm:PinHeader_1x05_P2.54mm_Vertical
- SW1, SW2, SW3, SW4: footprint Button_Switch_THT:SW_PUSH-12mm -> Button_Switch_THT:SW_PUSH_6mm
- renumbered H5 to H1, H6 to H2, H7 to H3, H8 to H4
Changed lines of the file:
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@@
   (symbol (lib_id "Mechanical:MountingHole_Pad") (at 72.39 124.46 0) (unit 1)
     (in_bom yes) (on_board yes) (dnp no) (fields_autoplaced)
-    (property "Reference" "H7" (at 74.93 121.92 0)
+    (property "Reference" "H3" (at 74.93 121.92 0)
       (effects (font (size 1.27 1.27)) (justify left))
     )
@@
       (project "dpad"
         (path "/050a8889-8bd8-4da8-9640-d64cfc084070"
-          (reference "H7") (unit 1)
+          (reference "H3") (unit 1)
         )
       )
@@
   (symbol (lib_id "Mechanical:MountingHole_Pad") (at 54.61 124.46 0) (unit 1)
     (in_bom yes) (on_board yes) (dnp no) (fields_autoplaced)
-    (property "Reference" "H5" (at 57.15 121.92 0)
+    (property "Reference" "H1" (at 57.15 121.92 0)
       (effects (font (size 1.27 1.27)) (justify left))
     )
@@
       (project "dpad"
         (path "/050a8889-8bd8-4da8-9640-d64cfc084070"
-          (reference "H5") (unit 1)
+          (reference "H1") (unit 1)
         )
       )
@@
   (symbol (lib_id "Mechanical:MountingHole_Pad") (at 63.5 124.46 0) (unit 1)
     (in_bom yes) (on_board yes) (dnp no) (fields_autoplaced)
-    (property "Reference" "H6" (at 66.04 121.92 0)
+    (property "Reference" "H2" (at 66.04 121.92 0)
       (effects (font (size 1.27 1.27)) (justify left))
     )
@@
       (project "dpad"
         (path "/050a8889-8bd8-4da8-9640-d64cfc084070"
-          (reference "H6") (unit 1)
+          (reference "H2") (unit 1)
         )
       )
@@
   (symbol (lib_id "Connector:Conn_01x05_Socket") (at 58.42 91.44 0) (unit 1)
     (in_bom yes) (on_board yes) (dnp no) (fields_autoplaced)
-    (property "Reference" "J6" (at 59.69 90.17 0)
+    (property "Reference" "J1" (at 59.69 90.17 0)
       (effects (font (size 1.27 1.27)) (justify left))
     )
@@
       (effects (font (size 1.27 1.27)) (justify left))
     )
-    (property "Footprint" "Connector_PinHeader_1.00mm:PinHeader_1x05_P1.00mm_Vertical" (at 58.42 91.44 0)
+    (property "Footprint" "Connector_PinHeader_2.54mm:PinHeader_1x05_P2.54mm_Vertical" (at 58.42 91.44 0)
       (effects (font (size 1.27 1.27)) hide)
     )
@@
       (project "dpad"
         (path "/050a8889-8bd8-4da8-9640-d64cfc084070"
-          (reference "J6") (unit 1)
+          (reference "J1") (unit 1)
         )
       )
@@
   (symbol (lib_id "Mechanical:MountingHole_Pad") (at 81.28 124.46 0) (unit 1)
     (in_bom yes) (on_board yes) (dnp no) (fields_autoplaced)
-    (property "Reference" "H8" (at 83.82 121.92 0)
+    (property "Reference" "H4" (at 83.82 121.92 0)
       (effects (font (size 1.27 1.27)) (justify left))
     )
@@
       (project "dpad"
         (path "/050a8889-8bd8-4da8-9640-d64cfc084070"
-          (reference "H8") (unit 1)
+          (reference "H4") (unit 1)
         )
       )
@@
       (effects (font (size 1.27 1.27)))
     )
-    (property "Footprint" "Button_Switch_THT:SW_PUSH-12mm" (at 59.69 50.8 0)
+    (property "Footprint" "Button_Switch_THT:SW_PUSH_6mm" (at 59.69 50.8 0)
       (effects (font (size 1.27 1.27)) hide)
     )
@@
       (effects (font (size 1.27 1.27)))
     )
-    (property "Footprint" "Button_Switch_THT:SW_PUSH-12mm" (at 93.98 50.8 0)
+    (property "Footprint" "Button_Switch_THT:SW_PUSH_6mm" (at 93.98 50.8 0)
       (effects (font (size 1.27 1.27)) hide)
     )
@@
       (effects (font (size 1.27 1.27)))
     )
-    (property "Footprint" "Button_Switch_THT:SW_PUSH-12mm" (at 76.2 67.31 0)
+    (property "Footprint" "Button_Switch_THT:SW_PUSH_6mm" (at 76.2 67.31 0)
       (effects (font (size 1.27 1.27)) hide)
     )
@@
       (effects (font (size 1.27 1.27)))
     )
-    (property "Footprint" "Button_Switch_THT:SW_PUSH-12mm" (at 77.47 36.83 0)
-      (effects (font (size 1.27 1.27)) hide)
-    )
+    (property "Footprint" "Button_Switch_THT:SW_PUSH_6mm" (at 77.47 36.83 0)
+      (effects (font (size 1.27 1.27)) hide)
+    )

Commit message: dpad v1
Parts:
- H1, H2, H3, H4: footprint MountingHole:MountingHole_3.2mm_M3_Pad -> MountingHole:MountingHole_2.2mm_M2_Pad
Other:
- company: (none) -> ALT.CTRL.GameCraft 2023
- title: Pico Controller -> D-Pad
Changed lines of the file:
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@@
   (paper "A4")
   (title_block
-    (title "Pico Controller")
-    (date "2023-09-17")
-    (rev "0")
+    (title "D-Pad")
+    (date "2023-09-26")
+    (rev "1")
+    (company "ALT.CTRL.GameCraft 2023")
   )
   (junction (at 72.39 127) (diameter 0) (color 0 0 0 0)
@@
       (effects (font (size 1.27 1.27)) (justify left))
     )
-    (property "Footprint" "MountingHole:MountingHole_3.2mm_M3_Pad" (at 72.39 124.46 0)
+    (property "Footprint" "MountingHole:MountingHole_2.2mm_M2_Pad" (at 72.39 124.46 0)
       (effects (font (size 1.27 1.27)) hide)
     )
@@
       (effects (font (size 1.27 1.27)) (justify left))
     )
-    (property "Footprint" "MountingHole:MountingHole_3.2mm_M3_Pad" (at 54.61 124.46 0)
+    (property "Footprint" "MountingHole:MountingHole_2.2mm_M2_Pad" (at 54.61 124.46 0)
       (effects (font (size 1.27 1.27)) hide)
     )
@@
       (effects (font (size 1.27 1.27)) (justify left))
     )
-    (property "Footprint" "MountingHole:MountingHole_3.2mm_M3_Pad" (at 63.5 124.46 0)
+    (property "Footprint" "MountingHole:MountingHole_2.2mm_M2_Pad" (at 63.5 124.46 0)
       (effects (font (size 1.27 1.27)) hide)
     )
@@
       (effects (font (size 1.27 1.27)) (justify left))
     )
-    (property "Footprint" "MountingHole:MountingHole_3.2mm_M3_Pad" (at 81.28 124.46 0)
-      (effects (font (size 1.27 1.27)) hide)
-    )
+    (property "Footprint" "MountingHole:MountingHole_2.2mm_M2_Pad" (at 81.28 124.46 0)
+      (effects (font (size 1.27 1.27)) hide)
+    )
